File: hardware/SteeringWheel.kicad_pcb (KiCad board)
At the start: 2 copper layers, 70 x 70 mm, 64 parts, among them SW1 SW_Push, SW10 SW_Push, SW7 SW_Push, SW8 SW_Push, SW9 SW_Push, U1 MCP2542FDxMF, U2 LMR36510ADDA, U3 LM3940, U4 STM32L4P5RETx, Y1 16MHz

Commit message: Placement done
Parts:
- removed C7, C8: 100nF, Capacitor_SMD:C_0603_1608Metric
- removed FB1: 60R@100MHz, Inductor_SMD:L_0603_1608Metric
- removed TP1: TestPoint_2Pole, TestPoint:TestPoint_2Pads_Pitch2.54mm_Drill0.8mm
- removed U1: MCP2542FDxMF, Package_DFN_QFN:DFN-8-1EP_3x3mm_P0.65mm_EP1.55x2.4mm
- added ?: , , F.Cu at (110.5, 130.5)
- added ?: , , F.Cu at (112.2, 70.0)
- added ?: , , F.Cu at (170.2, 71.0)
- added ?: , , F.Cu at (171.0, 129.5)
- added C19: 100n, Capacitor_SMD:C_0603_1608Metric, F.Cu at (137.6, 91.8)
- added C20: 100n, Capacitor_SMD:C_0603_1608Metric, F.Cu at (140.7, 86.5)
- added D1: PESD2IVN24-U, Package_TO_SOT_SMD:SOT-323_SC-70, F.Cu at (141.0, 94.7)
- added FB2: 470R, Inductor_SMD:L_0603_1608Metric, F.Cu at (137.6, 93.4)
- added FB3: 470R, Inductor_SMD:L_0603_1608Metric, F.Cu at (142.3, 86.5)
- added R5: 0R, Resistor_SMD:R_0603_1608Metric, F.Cu at (144.3, 91.8)
- added TP2: TestPoint_Small, TestPoint:TestPoint_Pad_D1.0mm, F.Cu at (144.8, 88.7)
- added TP3: TestPoint_Small, TestPoint:TestPoint_Pad_D1.0mm, F.Cu at (137.3, 88.6)
- added U5: MCP2542FD, Package_DFN_QFN:DFN-8-1EP_3x3mm_P0.65mm_EP1.55x2.4mm, F.Cu at (141.0, 90.2)
- L2: footprint Inductor_SMD:L_7.3x7.3_H4.5 -> Inductor_SMD:L_0603_1608Metric
- SW1: footprint KiCad:7914J1000E -> Button_Switch_SMD:SW_SPST_B3U-1000P
- Y1: footprint Crystal:Crystal_SMD_2520-4Pin_2.5x2.0mm -> Crystal:Crystal_SMD_Abracon_ABM8G-4Pin_3.2x2.5mm
- moved C11 112.4 mm to (168.1, 89.3), turned to 90 degrees
- moved C14 111.3 mm to (167.7, 101.0)
- moved C33 107.8 mm to (165.2, 84.0)
- moved SW7 103.6 mm to (162.9, 80.3), turned to 180 degrees
- moved R4 103.0 mm to (161.4, 87.5), turned to 180 degrees
- moved C10 101.3 mm to (157.1, 88.2), turned to 90 degrees
- moved R30 101.0 mm to (162.1, 84.0)
- moved R13 100.5 mm to (166.2, 111.1), turned to 90 degrees
- moved C18 99.4 mm to (160.3, 120.5)
- moved C9 99.1 mm to (155.5, 89.3), turned to 90 degrees
- moved C34 98.7 mm to (155.8, 84.0)
- moved R14 98.6 mm to (164.4, 111.1), turned to 90 degrees
- moved C31 98.5 mm to (160.2, 102.5)
- moved C12 98.2 mm to (153.2, 90.6), turned to 180 degrees
- moved C13 97.8 mm to (153.6, 96.4)
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Connections:
- U4 pad 12: Net-(U4-VSSA) -> GND
- U4 pad 18: Net-(U4-VSSA) -> GND
- U4 pad 31: Net-(U4-VSSA) -> GND
- U4 pad 47: Net-(U4-VSSA) -> GND
- U4 pad 63: Net-(U4-VSSA) -> GND

Commit message: Layout done
Parts:
- added J2: FTSH, ftsh-107-01-l-dv-k-a:FTSH-107-XX-YYY-DV-K-A, F.Cu at (155.2, 108.6)
- D5: footprint Diode_SMD:D_MELF -> Diode_SMD:D_SOD-123
- moved G*** 105.9 mm to (126.0, 128.0)
- moved G*** 98.7 mm to (126.0, 128.0)
- moved C18 36.8 mm to (125.0, 110.3), turned to 90 degrees
- moved SW1 34.4 mm to (122.5, 113.9), turned to -90 degrees
- moved R12 33.1 mm to (125.0, 113.3), turned to 90 degrees
- moved C14 32.6 mm to (142.5, 121.8), turned to 180 degrees
- moved C31 30.9 mm to (136.0, 121.7), turned to 180 degrees
- moved C11 30.2 mm to (146.8, 110.8), turned to -90 degrees
- moved C32 29.9 mm to (131.6, 118.0)
- moved C9 29.9 mm to (132.6, 108.5)
- moved L2 29.9 mm to (130.0, 118.0)
- moved R4 29.9 mm to (138.5, 106.7)
- moved U4 29.9 mm to (139.1, 114.2)
- moved C13 29.9 mm to (130.7, 115.6)
- moved Y1 29.8 mm to (130.6, 112.6)
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Connections:
- U4 pad 46: unconnected-(U4-PA13-Pad46) -> /SWDIO
- U4 pad 49: unconnected-(U4-PA14-Pad49) -> /SWCLK
Routing:
- net +3.3V: track 2.87 -> 209.6 mm, vias 0 -> 8
- net /CAN_RX: track 0.00 -> 78.0 mm, vias 0 -> 2
- net /sw3: track 0.00 -> 61.5 mm, vias 0 -> 2
- net /sw2: track 0.00 -> 57.0 mm
- net /sw1: track 0.00 -> 56.3 mm
- net /sw4: track 0.00 -> 54.3 mm, vias 0 -> 2
- net /CAN_TX: track 0.00 -> 52.8 mm, vias 0 -> 2
- net /NRST: track 0.00 -> 49.6 mm, vias 0 -> 3
- net /SWDIO: track 0.00 -> 23.6 mm, vias 0 -> 2
- net /SWCLK: track 0.00 -> 22.5 mm, vias 0 -> 2
- net +5V: track 33.8 -> 55.4 mm, vias 3 -> 5
- net /LED2: track 0.00 -> 11.7 mm
- net /LED4: track 0.00 -> 11.4 mm, vias 0 -> 2
- net /CAN_L: track 0.00 -> 10.9 mm
- net /CAN_H: track 0.00 -> 10.9 mm, vias 0 -> 1
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- added copper zone on B.Cu, net +3.3V
- added copper zone on F.Cu, net +3.3V
Other:
- board text added: "Steering Wheel"
- board text removed: "made by Tadeusz Zakola"

Commit message: Vias and adnotations update
Routing:
- net GND: vias 2 -> 419

Commit message: Fix minor issues
Parts:
- added JP1: JP Open, Jumper:SolderJumper-2_P1.3mm_Open_Pad1.0x1.5mm, F.Cu at (144.0, 78.5)
- added R6: 120R, Resistor_SMD:R_0603_1608Metric, F.Cu at (144.0, 80.5)
- added TP1: TestPoint_Small, TestPoint:TestPoint_Pad_D1.0mm, F.Cu at (133.5, 120.0)
- added TP4: TestPoint_Small, TestPoint:TestPoint_Pad_D1.0mm, F.Cu at (138.0, 124.0)
- added TP5: TestPoint_Small, TestPoint:TestPoint_Pad_D1.0mm, F.Cu at (139.5, 125.5)
- added TP6: TestPoint_Small, TestPoint:TestPoint_Pad_D1.0mm, F.Cu at (141.0, 124.0)
- added TP7: TestPoint_Small, TestPoint:TestPoint_Pad_D1.0mm, F.Cu at (142.5, 125.5)
- C16: value 100nF -> 1uF
- moved C31 0.77 mm to (136.0, 122.5), turned to -90 degrees
Connections:
- U4 pad 17: unconnected-(U4-PA3-Pad17) -> Net-(U4-PA3)
- U4 pad 20: unconnected-(U4-PA4-Pad20) -> Net-(U4-PA4)
- U4 pad 21: unconnected-(U4-PA5-Pad21) -> Net-(U4-PA5)
- U4 pad 22: unconnected-(U4-PA6-Pad22) -> Net-(U4-PA6)
- U4 pad 23: unconnected-(U4-PA7-Pad23) -> Net-(U4-PA7)
Routing:
- net Net-(U4-PA7): track 0.00 -> 7.93 mm
- net Net-(U4-PA5): track 0.00 -> 6.48 mm
- net Net-(U4-PA6): track 0.00 -> 5.98 mm
- net Net-(U4-PA4): track 0.00 -> 4.57 mm
- net +3.3V: track 209.6 -> 212.9 mm, vias 8 -> 9
- net /CAN_L: track 10.9 -> 13.3 mm
- net /CAN_H: track 10.9 -> 13.0 mm
- net Net-(JP1-A): track 0.00 -> 2.07 mm
- net Net-(U4-PA3): track 0.00 -> 1.89 mm
- net GND: track 8.54 -> 7.68 mm, vias 419 -> 410
- net +5V: vias 5 -> 4
